File: hardware/rev0.1/RFIDetector.kicad_pcb (KiCad board)
At the start: 4 copper layers, 49.8 x 49.8 mm, 41 parts

Commit message: Rev 0.1
Parts:
- C13, C14, C15, C16, C18, C19, C20, C21, C22, C23: value C -> 0
- C17: value C -> 4.7n
Changed lines of the file:
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@@
   )
   (paper "A4")
+  (title_block
+    (title "RFIDetector")
+    (rev "0.1")
+    (company "wh201906")
+  )
   (layers
     (0 "F.Cu" signal)
@@
         (effects (font (size 1 1) (thickness 0.15)) (justify top))
     )
-    (fp_text value "C" (at 0 1.43) (layer "F.Fab")
+    (fp_text value "4.7n" (at 0 1.43) (layer "F.Fab")
         (effects (font (size 1 1) (thickness 0.15)))
     )
@@
         (effects (font (size 1 1) (thickness 0.15)) (justify top))
     )
-    (fp_text value "C" (at 0 1.43) (layer "F.Fab")
+    (fp_text value "0" (at 0 1.43) (layer "F.Fab")
         (effects (font (size 1 1) (thickness 0.15)))
     )
@@
         (effects (font (size 1 1) (thickness 0.15)) (justify top))
     )
-    (fp_text value "C" (at 0 1.43) (layer "F.Fab")
+    (fp_text value "0" (at 0 1.43) (layer "F.Fab")
         (effects (font (size 1 1) (thickness 0.15)))
     )
@@
         (effects (font (size 1 1) (thickness 0.15)) (justify top))
     )
-    (fp_text value "C" (at 0 1.43) (layer "F.Fab")
+    (fp_text value "0" (at 0 1.43) (layer "F.Fab")
         (effects (font (size 1 1) (thickness 0.15)))
     )
@@
         (effects (font (size 1 1) (thickness 0.15)) (justify top))
     )
-    (fp_text value "C" (at 0 1.43) (layer "F.Fab")
+    (fp_text value "0" (at 0 1.43) (layer "F.Fab")
         (effects (font (size 1 1) (thickness 0.15)))
     )
@@
         (effects (font (size 1 1) (thickness 0.15)) (justify top))
     )
-    (fp_text value "C" (at 0 1.43) (layer "F.Fab")
+    (fp_text value "0" (at 0 1.43) (layer "F.Fab")
         (effects (font (size 1 1) (thickness 0.15)))
     )
@@
         (effects (font (size 1 1) (thickness 0.15)) (justify top))
     )
-    (fp_text value "C" (at 0.6 1.4625) (layer "F.Fab")
+    (fp_text value "0" (at 0.6 1.4625) (layer "F.Fab")
         (effects (font (size 1 1) (thickness 0.15)))
     )
@@
         (effects (font (size 1 1) (thickness 0.15)) (justify top))
     )
-    (fp_text value "C" (at 0.01 1.43) (layer "F.Fab")
+    (fp_text value "0" (at 0.01 1.43) (layer "F.Fab")
         (effects (font (size 1 1) (thickness 0.15)))
     )
@@
         (effects (font (size 1 1) (thickness 0.15)) (justify top))
     )
-    (fp_text value "C" (at 0 1.43) (layer "F.Fab")
+    (fp_text value "0" (at 0 1.43) (layer "F.Fab")
         (effects (font (size 1 1) (thickness 0.15)))
     )
@@
         (effects (font (size 1 1) (thickness 0.15)) (justify top))
     )
-    (fp_text value "C" (at -0.08 1.48) (layer "F.Fab")
+    (fp_text value "0" (at -0.08 1.48) (layer "F.Fab")
         (effects (font (size 1 1) (thickness 0.15)))
     )
@@
         (effects (font (size 1 1) (thickness 0.15)) (justify top))
     )
-    (fp_text value "C" (at 0 1.43) (layer "F.Fab")
-        (effects (font (size 1 1) (thickness 0.15)))
-    )
+    (fp_text value "0" (at 0 1.43) (layer "F.Fab")
+        (effects (font (size 1 1) (thickness 0.15)))
+    )
