File: hardware/rev0.1/RFIDetector.kicad_sch (KiCad schematic)
At the start: 41 parts

Commit message: Rev 0.1
Parts:
- C13, C14, C15, C16, C18, C19, C20, C21, C22, C23: value C -> 0
- C17: value C -> 4.7n
Other:
- company: (none) -> wh201906
- title: (none) -> RFIDetector
Changed lines of the file:
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@@
 (kicad_sch (version 20230121) (generator eeschema)
   (paper "A4")
+  (title_block
+    (title "RFIDetector")
+    (rev "0.1")
+    (company "wh201906")
+  )
   (junction (at 95.25 58.42) (diameter 0) (color 0 0 0 0)
   )
@@
       (effects (font (size 1.27 1.27)) (justify right))
     )
-    (property "Value" "C" (at 220.091 57.0921 0)
+    (property "Value" "0" (at 220.091 57.0921 0)
       (effects (font (size 1.27 1.27)) (justify right))
     )
@@
       (effects (font (size 1.27 1.27)) (justify left))
     )
-    (property "Value" "C" (at 189.611 129.4821 0)
+    (property "Value" "0" (at 189.611 129.4821 0)
       (effects (font (size 1.27 1.27)) (justify left))
     )
@@
       (effects (font (size 1.27 1.27)) (justify right))
     )
-    (property "Value" "C" (at 199.771 57.0921 0)
+    (property "Value" "4.7n" (at 199.771 57.0921 0)
       (effects (font (size 1.27 1.27)) (justify right))
     )
@@
       (effects (font (size 1.27 1.27)) (justify right))
     )
-    (property "Value" "C" (at 179.451 57.0921 0)
+    (property "Value" "0" (at 179.451 57.0921 0)
       (effects (font (size 1.27 1.27)) (justify right))
     )
@@
       (effects (font (size 1.27 1.27)) (justify left))
     )
-    (property "Value" "C" (at 179.451 139.6421 0)
+    (property "Value" "0" (at 179.451 139.6421 0)
       (effects (font (size 1.27 1.27)) (justify left))
     )
@@
       (effects (font (size 1.27 1.27)) (justify right))
     )
-    (property "Value" "C" (at 209.931 57.0921 0)
+    (property "Value" "0" (at 209.931 57.0921 0)
       (effects (font (size 1.27 1.27)) (justify right))
     )
@@
       (effects (font (size 1.27 1.27)) (justify left))
     )
-    (property "Value" "C" (at 199.771 129.4821 0)
+    (property "Value" "0" (at 199.771 129.4821 0)
       (effects (font (size 1.27 1.27)) (justify left))
     )
@@
       (effects (font (size 1.27 1.27)) (justify left))
     )
-    (property "Value" "C" (at 189.611 57.0921 0)
+    (property "Value" "0" (at 189.611 57.0921 0)
       (effects (font (size 1.27 1.27)) (justify left))
     )
@@
       (effects (font (size 1.27 1.27)) (justify right))
     )
-    (property "Value" "C" (at 179.451 129.4821 0)
+    (property "Value" "0" (at 179.451 129.4821 0)
       (effects (font (size 1.27 1.27)) (justify right))
     )
@@
       (effects (font (size 1.27 1.27)) (justify left))
     )
-    (property "Value" "C" (at 179.451 67.2521 0)
+    (property "Value" "0" (at 179.451 67.2521 0)
       (effects (font (size 1.27 1.27)) (justify left))
     )
@@
       (effects (font (size 1.27 1.27)) (justify left))
     )
-    (property "Value" "C" (at 189.611 67.2521 0)
-      (effects (font (size 1.27 1.27)) (justify left))
-    )
+    (property "Value" "0" (at 189.611 67.2521 0)
+      (effects (font (size 1.27 1.27)) (justify left))
+    )
